File: KiCAD PCB Design/LTC1871_Boost_FYP_KiCad/LTC1871_Based_Boost_Controller/LTC1871_Based_Boost_Controller.kicad_sch (KiCad schematic)
At the start: 29 parts, among them J2 J2_OUT, Q1 IRF7811, U1 LTC1871EMS-7-PBF

Commit message: Auto-sync from Fortune at 2026-04-08 21:37:35
Parts:
- J2: footprint (none) -> Connector_PinHeader_2.54mm:PinHeader_1x02_P2.54mm_Vertical
Changed lines of the file:
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@@
 			)
 		)
-		(property "Footprint" ""
+		(property "Footprint" "Connector_PinHeader_2.54mm:PinHeader_1x02_P2.54mm_Vertical"
 			(at 269.24 67.31 0)
 			(hide yes)

Commit message: Auto-sync from Fortune at 2026-04-09 18:59:21
Parts:
- added Q2: DMP3099L, Package_TO_SOT_SMD:SOT-23, symbol Transistor_FET:Q_PMOS_GSD
- added R5: 549k, Resistor_SMD:R_0805_2012Metric, symbol Device:R
- added R6: 100K, Resistor_SMD:R_0805_2012Metric, symbol Device:R
Connections:
- net GND: now also Q2.1 (G), R6.2
- net at C6.1, C7.1, Cin1.1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: now also Q2.2 (S), Q2.3 (D), R5.1; no longer D1.1 (K), L1.2, Q1.2 (D), U1.1 (RUN), U1.10 (SENSE)
- new net: D1.1 (K), L1.2, Q1.2 (D), Q1.4 (Drain), Q1.5 (Drain), Q1.6 (Drain), Q1.7 (Drain), Q1.8 (Drain), U1.10 (SENSE)
- new net: R5.2, R6.1, U1.1 (RUN)
Other:
- moved on the sheet: C1, C2, C3, D2, Q1, R4

Commit message: Auto-sync from Fortune at 2026-04-10 15:43:13
Parts:
- added J3: Proto_GND, Connector_PinHeader_2.54mm:PinHeader_1x05_P2.54mm_Vertical, symbol Connector_Generic:Conn_01x05
- added J4: Proto_1, Connector_PinHeader_2.54mm:PinHeader_1x05_P2.54mm_Vertical, symbol Connector_Generic:Conn_01x05
- added J5: Proto_2, Connector_PinHeader_2.54mm:PinHeader_1x05_P2.54mm_Vertical, symbol Connector_Generic:Conn_01x05
Connections:
- net GND: now also J3.1 (Pin_1), J4.1 (Pin_1), J5.1 (Pin_1)
- net at C6.1, C7.1, Cin1.1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: now also J4.2 (Pin_2)
- net at C1a1.1, C1a2.1, C1a3.1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: now also J5.2 (Pin_2)

Commit message: Auto-sync from Fortune at 2026-04-11 22:57:18
Parts:
- Q1: value IRF7811 -> SQ4184EY
Connections:
- no-connect marks 0 -> 10
Changed lines of the file:
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@@
 		(color 0 0 0 0)
 	)
+	(no_connect
+		(at 52.07 160.02)
+	)
+	(no_connect
+		(at 91.44 147.32)
+	)
+	(no_connect
+		(at 52.07 133.35)
+	)
+	(no_connect
+		(at 91.44 152.4)
+	)
+	(no_connect
+		(at 52.07 162.56)
+	)
+	(no_connect
+		(at 52.07 165.1)
+	)
+	(no_connect
+		(at 52.07 125.73)
+	)
+	(no_connect
+		(at 91.44 149.86)
+	)
+	(no_connect
+		(at 52.07 128.27)
+	)
+	(no_connect
+		(at 52.07 130.81)
+	)
 	(wire
 		(pts
@@
 			)
 		)
-		(property "Value" "IRF7811"
+		(property "Value" "SQ4184EY"
 			(at 165.1 97.7899 0)
 			(show_name no)

Commit message: Auto-sync from Fortune at 2026-04-13 06:50:55
Parts:
- Q1: value SQ4184EY -> SI4894BDY
Changed lines of the file:
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@@
 			)
 		)
-		(property "Value" "SQ4184EY"
+		(property "Value" "SI4894BDY"
 			(at 165.1 97.7899 0)
 			(show_name no)
