File: KiCAD PCB Design/LTC1871_Boost_FYP_KiCad/LTC1871_Based_Boost_Controller/LTC1871_Based_Boost_Controller.kicad_pcb (KiCad board)
At the start: 2 copper layers, 29 parts, among them J2 J2_OUT, Q1 IRF7811, U1 LTC1871EMS-7-PBF

Commit message: Auto-sync from Fortune at 2026-04-08 23:37:36
Parts:
- moved J_VIN1 151.4 mm to (14.0, 22.9), turned to 90 degrees
- moved C1b1 137.8 mm to (22.9, 20.3), turned to 90 degrees
- moved C1b2 136.5 mm to (22.9, 25.4), turned to 90 degrees
- moved Q1 130.7 mm to (34.3, 34.3)
- moved L1 130.3 mm to (34.3, 22.9)
- moved Cin1 126.8 mm to (16.5, 36.8)
- moved C5 115.8 mm to (16.5, 50.8)
- moved J2 111.2 mm to (65.9, 19.1), turned to 90 degrees
- moved R1 111.0 mm to (26.7, 76.2)
- moved C2 110.5 mm to (26.7, 62.2)
- moved D2 107.1 mm to (26.7, 68.6)
- moved D1 101.7 mm to (52.1, 14.0)
- moved C1 101.1 mm to (35.6, 62.2)
- moved C3 99.0 mm to (35.6, 76.2)
- moved R3 98.8 mm to (44.5, 62.2)
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Routing:
- net Net-(D1-K): track 0.00 -> 160.9 mm
- net Net-(D1-A): track 0.00 -> 144.3 mm, vias 0 -> 1
- net Net-(Q1-G): track 0.00 -> 48.2 mm
- net Net-(D2-K): track 0.00 -> 41.3 mm
- net GND: track 0.00 -> 40.8 mm, vias 0 -> 21
- net Net-(C2-Pad1): track 0.00 -> 26.3 mm, vias 0 -> 2
- net Net-(U1-FB): track 0.00 -> 18.6 mm
- net Net-(U1-INTVCC): track 0.00 -> 14.3 mm
- net Net-(U1-FREQ): track 0.00 -> 10.0 mm
- net Net-(D2-A): track 0.00 -> 5.75 mm
- added copper zone on B.Cu, net GND
Other:
- board outline added: 60 x 80 mm
- board text added: "LTC1871 Boost Controller"
- board text added: "VIN 8-12V"
- board text added: "VOUT 12V"

Commit message: Auto-sync from Fortune at 2026-04-08 23:49:32
Parts:
- removed C1: 10n, Capacitor_SMD:C_0805_2012Metric
- removed C1a1, C1a2, C1a3, C1a4, C1a5, C1a6, C1a7, C1a8, C6, C7: 22µ, Capacitor_SMD:C_1206_3216Metric
- removed C1b1, C1b2: 10µ, Capacitor_SMD:C_0805_2012Metric
- removed C2: 6.8n, Capacitor_SMD:C_0805_2012Metric
- removed C3: 100p, Capacitor_SMD:C_0805_2012Metric
- removed C4: 4.7µ, Capacitor_SMD:C_0805_2012Metric
- removed C5, Cin1: 100µ, Capacitor_THT:CP_Radial_D8.0mm_P3.50mm
- removed D1: MBR735, Diode_THT:D_DO-201AD_P15.24mm_Horizontal
- removed D2: 1N4148, Diode_SMD:D_SOD-323_HandSoldering
- removed J2: J2_OUT, Connector_PinHeader_2.54mm:PinHeader_1x02_P2.54mm_Vertical
- removed J_VIN1: J_VIN_OUT, Connector_PinHeader_2.54mm:PinHeader_1x02_P2.54mm_Vertical
- removed L1: 10µ, Inductor_SMD:L_Coilcraft_XAL6060-XXX
- removed Q1: IRF7811, Package_SO:SOIC-8_3.9x4.9mm_P1.27mm
- removed R1: 68.1k, Resistor_SMD:R_0805_2012Metric
- removed R2: 56k, Resistor_SMD:R_0805_2012Metric
- removed R3: 499k, Resistor_SMD:R_0805_2012Metric
- removed R4: 8.66k, Resistor_SMD:R_0805_2012Metric
- removed U1: LTC1871EMS-7-PBF, Package_SO:MSOP-10_3x3mm_P0.5mm
Routing:
- net Net-(D1-K): track 160.9 -> 0.00 mm
- net Net-(D1-A): track 144.3 -> 0.00 mm, vias 1 -> 0
- net Net-(Q1-G): track 48.2 -> 0.00 mm
- net Net-(D2-K): track 41.3 -> 0.00 mm
- net GND: track 40.8 -> 0.06 mm, vias 21 -> 0
- net Net-(C2-Pad1): track 26.3 -> 0.00 mm, vias 2 -> 0
- net Net-(U1-FB): track 18.6 -> 0.00 mm
- net Net-(U1-INTVCC): track 14.3 -> 0.00 mm
- net Net-(U1-FREQ): track 10.0 -> 0.00 mm
- net Net-(D2-A): track 5.75 -> 0.00 mm
- removed copper zone on B.Cu, net GND
Other:
- board outline removed
- board text removed: "LTC1871 Boost Controller"
- board text removed: "VIN 8-12V"
- board text removed: "VOUT 12V"

Commit message: Auto-sync from Fortune at 2026-04-09 18:59:21
Parts:
- added C1: 10n, Capacitor_SMD:C_0805_2012Metric, F.Cu at (193.5, 136.5)
- added C1a1: 22µ, Capacitor_SMD:C_1206_3216Metric, F.Cu at (224.0, 115.0)
- added C1a2: 22µ, Capacitor_SMD:C_1206_3216Metric, F.Cu at (224.0, 118.3)
- added C1a3: 22µ, Capacitor_SMD:C_1206_3216Metric, F.Cu at (224.0, 121.7)
- added C1a4: 22µ, Capacitor_SMD:C_1206_3216Metric, F.Cu at (224.0, 125.0)
- added C1a5: 22µ, Capacitor_SMD:C_1206_3216Metric, F.Cu at (224.0, 128.3)
- added C1a6: 22µ, Capacitor_SMD:C_1206_3216Metric, F.Cu at (224.0, 131.7)
- added C1a7: 22µ, Capacitor_SMD:C_1206_3216Metric, F.Cu at (224.0, 135.1)
- added C1a8: 22µ, Capacitor_SMD:C_1206_3216Metric, F.Cu at (224.0, 138.4)
- added C1b1: 10µ, Capacitor_SMD:C_0805_2012Metric, F.Cu at (228.5, 108.0)
- added C1b2: 10µ, Capacitor_SMD:C_0805_2012Metric, F.Cu at (228.5, 111.0)
- added C2: 6.8n, Capacitor_SMD:C_0805_2012Metric, F.Cu at (193.5, 139.5)
- added C3: 100p, Capacitor_SMD:C_0805_2012Metric, F.Cu at (193.5, 142.5)
- added C4: 4.7µ, Capacitor_SMD:C_0805_2012Metric, F.Cu at (211.5, 130.0)
- added C5: 100µ, Capacitor_THT:CP_Radial_D8.0mm_P3.50mm, F.Cu at (177.8, 138.5)
- added C6: 22µ, Capacitor_SMD:C_1206_3216Metric, F.Cu at (176.0, 109.0)
- added C7: 22µ, Capacitor_SMD:C_1206_3216Metric, F.Cu at (179.0, 109.0)
- added Cin1: 100µ, Capacitor_THT:CP_Radial_D8.0mm_P3.50mm, F.Cu at (185.5, 129.0)
- added D1: MBR735, Diode_THT:D_DO-201AD_P15.24mm_Horizontal, F.Cu at (213.5, 126.6)
- added D2: 1N4148, Diode_SMD:D_SOD-323_HandSoldering, F.Cu at (203.2, 136.0)
- added J2: J2_OUT, Connector_PinHeader_2.54mm:PinHeader_1x02_P2.54mm_Vertical, F.Cu at (231.5, 126.0)
- added J_VIN1: J_VIN_OUT, Connector_PinHeader_2.54mm:PinHeader_1x02_P2.54mm_Vertical, F.Cu at (178.5, 120.5)
- added L1: 10µ, Inductor_SMD:L_Coilcraft_XAL6060-XXX, F.Cu at (194.5, 121.0)
- added Q1: IRF7811, Package_SO:SOIC-8_3.9x4.9mm_P1.27mm, F.Cu at (204.5, 120.4)
- added Q2: DMP3099L, Package_TO_SOT_SMD:SOT-23, F.Cu at (186.1, 122.0)
- added R1: 68.1k, Resistor_SMD:R_0805_2012Metric, F.Cu at (207.0, 140.0)
- added R2: 56k, Resistor_SMD:R_0805_2012Metric, F.Cu at (212.6, 134.0)
- added R3: 499k, Resistor_SMD:R_0805_2012Metric, F.Cu at (212.6, 136.9)
- added R4: 8.66k, Resistor_SMD:R_0805_2012Metric, F.Cu at (193.6, 134.0)
- added R5: 549k, Resistor_SMD:R_0805_2012Metric, F.Cu at (184.1, 112.0)
- added R6: 100K, Resistor_SMD:R_0805_2012Metric, F.Cu at (184.1, 115.0)
- added U1: LTC1871EMS-7-PBF, Package_SO:MSOP-10_3x3mm_P0.5mm, F.Cu at (203.5, 129.0)
Routing:
- net GND: track 0.06 -> 315.5 mm, vias 0 -> 16
- net Net-(D1-A): track 0.00 -> 110.0 mm
- net Net-(J_VIN1-Pin_1): track 0.00 -> 107.8 mm
- net Net-(D1-K): track 0.00 -> 37.5 mm
- net Net-(Q1-G): track 0.00 -> 24.9 mm
- net Net-(U1-FB): track 0.00 -> 16.6 mm
- net Net-(D2-K): track 0.00 -> 15.5 mm
- net Net-(U1-FREQ): track 0.00 -> 14.5 mm
- net Net-(D2-A): track 0.00 -> 10.4 mm
- net Net-(U1-INTVCC): track 0.00 -> 6.94 mm
- net Net-(C2-Pad1): track 0.00 -> 6.29 mm
- net Net-(U1-RUN): track 0.00 -> 4.14 mm
- added copper zone on B.Cu, net GND
Other:
- board outline added: 59.5 x 40 mm

Commit message: Auto-sync from Fortune at 2026-04-09 20:51:06
Routing:
- net GND: track 315.5 -> 0.00 mm, vias 16 -> 0
- net Net-(D1-A): track 110.0 -> 0.00 mm
- net Net-(J_VIN1-Pin_1): track 107.8 -> 0.00 mm
- net Net-(D1-K): track 37.5 -> 0.00 mm
- net Net-(Q1-G): track 24.9 -> 0.00 mm
- net Net-(U1-FB): track 16.6 -> 0.00 mm
- net Net-(D2-K): track 15.5 -> 0.00 mm
- net Net-(U1-FREQ): track 14.5 -> 0.00 mm
- net Net-(D2-A): track 10.4 -> 0.00 mm
- net Net-(U1-INTVCC): track 6.94 -> 0.00 mm
- net Net-(C2-Pad1): track 6.29 -> 0.00 mm
- net Net-(U1-RUN): track 4.14 -> 0.00 mm

Commit message: Auto-sync from Fortune at 2026-04-10 00:15:56
Parts:
- moved C5 41.6 mm to (206.0, 107.8), turned to -90 degrees
- moved Cin1 23.7 mm to (195.5, 107.5)
- moved R3 5.73 mm to (208.1, 140.5)
- moved R4 5.59 mm to (199.1, 133.0)
- moved R1 5.58 mm to (201.5, 140.9), turned to 90 degrees
- moved R2 5.10 mm to (207.6, 135.0)
- moved C1 4.00 mm to (197.5, 136.5), turned to -90 degrees
- moved C2 3.14 mm to (190.5, 140.4), turned to -90 degrees
- moved C3 2.95 mm to (196.0, 140.9), turned to 90 degrees
- moved C6 2.60 mm to (176.5, 111.5)
- moved C4 2.50 mm to (209.1, 129.5)
- moved Q2 1.72 mm to (184.4, 121.5)
- moved R5 1.10 mm to (185.1, 112.5)
- moved C7 1.00 mm to (180.0, 109.0)
- moved R6 1.00 mm to (185.1, 115.0)
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Routing:
- net Net-(D1-A): track 0.00 -> 94.5 mm
- net Net-(J_VIN1-Pin_1): track 0.00 -> 94.1 mm
- net Net-(U1-RUN): track 0.00 -> 68.3 mm, vias 0 -> 2
- net Net-(D1-K): track 0.00 -> 50.3 mm, vias 0 -> 1
- net Net-(D2-K): track 0.00 -> 47.4 mm, vias 0 -> 7
- net Net-(U1-FB): track 0.00 -> 32.2 mm
- net Net-(Q1-G): track 0.00 -> 30.0 mm
- net GND: track 0.00 -> 20.1 mm, vias 0 -> 3
- net Net-(U1-FREQ): track 0.00 -> 11.8 mm
- net Net-(C2-Pad1): track 0.00 -> 10.4 mm
- net Net-(D2-A): track 0.00 -> 8.53 mm
- net Net-(U1-INTVCC): track 0.00 -> 6.12 mm

Commit message: Auto-sync from Fortune at 2026-04-10 15:43:13
Parts:
- added J3: Proto_GND, Connector_PinHeader_2.54mm:PinHeader_1x05_P2.54mm_Vertical, F.Cu at (176.8, 130.8)
- added J4: Proto_1, Connector_PinHeader_2.54mm:PinHeader_1x05_P2.54mm_Vertical, F.Cu at (181.4, 130.8)
- added J5: Proto_2, Connector_PinHeader_2.54mm:PinHeader_1x05_P2.54mm_Vertical, F.Cu at (186.0, 130.8)
Routing:
- net GND: track 20.1 -> 381.0 mm, vias 3 -> 13
- net Net-(U1-INTVCC): track 6.12 -> 43.3 mm, vias 0 -> 3
- net Net-(D1-A): track 94.5 -> 130.3 mm
- net Net-(J4-Pin_2): track 94.1 -> 109.9 mm, vias 0 -> 1

Commit message: Auto-sync from Fortune at 2026-04-10 17:12:48
Parts:
- moved C4 73.3 mm to (142.1, 99.6)
- moved R5 73.3 mm to (118.2, 82.6)
- moved R6 73.3 mm to (118.2, 85.1)
- moved C1 73.3 mm to (130.6, 106.6)
- moved C1a1 73.3 mm to (157.1, 85.0)
- moved C1a2 73.3 mm to (157.1, 88.4)
- moved C1a3 73.3 mm to (157.1, 91.8)
- moved C1a4 73.3 mm to (157.1, 95.1)
- moved C1a5 73.3 mm to (157.1, 98.5)
- moved C1a6 73.3 mm to (157.1, 101.8)
- moved C1a7 73.3 mm to (157.1, 105.2)
- moved C1a8 73.3 mm to (157.1, 108.5)
- moved C1b1 73.3 mm to (161.6, 78.1)
- moved C1b2 73.3 mm to (161.6, 81.1)
- moved C2 73.3 mm to (123.6, 110.5)
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