File: KiCAD PCB Design/LTC1871_Boost_FYP_KiCad/LTC1871_Based_Boost_Controller/LTC1871_Based_Boost_Controller.kicad_pcb (KiCad board)
At the start: 2 copper layers, 59.5 x 40 mm, 35 parts, among them J2 J2_OUT, J3 Proto_GND, J4 Proto_1, J5 Proto_2, Q1 IRF7811, Q2 DMP3099L, U1 LTC1871EMS-7-PBF

Commit message: Auto-sync from Fortune at 2026-04-11 22:57:18
Parts:
- Q1: value IRF7811 -> SQ4184EY
- moved C1 0.71 mm to (131.1, 107.1)
- moved C1a1 0.71 mm to (157.6, 85.5)
- moved C1a2 0.71 mm to (157.6, 88.9)
- moved C1a3 0.71 mm to (157.6, 92.2)
- moved C1a4 0.71 mm to (157.6, 95.6)
- moved C1a5 0.71 mm to (157.6, 99.0)
- moved C1a6 0.71 mm to (157.6, 102.3)
- moved C1a7 0.71 mm to (157.6, 105.7)
- moved C1a8 0.71 mm to (157.6, 109.0)
- moved C1b1 0.71 mm to (162.1, 78.6)
- moved C1b2 0.71 mm to (162.1, 81.6)
- moved C2 0.71 mm to (124.1, 111.0)
- moved C3 0.71 mm to (129.6, 111.5)
- moved C4 0.71 mm to (142.6, 100.1)
- moved C5 0.71 mm to (139.6, 78.4)
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Routing:
- added copper zone on F.Cu, net GND

Commit message: Auto-sync from Fortune at 2026-04-13 21:30:20
Parts:
- added C8: 220n, Capacitor_SMD:C_0805_2012Metric, F.Cu at (124.2, 97.0)
- Q1: value SQ4184EY -> SI4894BDY
Routing:
- net Net-(C2-Pad1): track 10.4 -> 26.6 mm, vias 0 -> 2
- net GND: track 381.0 -> 391.0 mm, vias 13 -> 14
