File: KiCAD PCB Design/LTC1871_Based_Boost_Controller/LTC1871_Based_Boost_Controller.kicad_pcb (KiCad board)
At the start: 2 copper layers, 29 parts, among them J2 J2_OUT, Q1 IRF7811, U1 LTC1871EMS-7-PBF

Commit message: Auto-sync from Fortune at 2026-04-09 08:51:17
Parts:
- moved C5 0.53 mm to (123.3, 95.0)
Changed lines of the file:
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@@
 	(footprint "Capacitor_THT:CP_Radial_D8.0mm_P3.50mm"
 		(layer "F.Cu")
-		(at 123.369698 95.525)
+		(at 123.347349 95)
 		(descr "CP, Radial series, Radial, pin pitch=3.50mm, diameter=8mm, height=12mm, Electrolytic Capacitor")
 		(tags "CP Radial series Radial pin pitch 3.50mm diameter 8mm height 12mm Electrolytic Capacitor")
