File: KiCAD PCB Design/LTC1871 KiCAD PCD Revision/LTC1871_Based_Boost_Controller_V2.kicad_pcb (KiCad board)
At the start: 2 copper layers, 60.5 x 42.5 mm, 36 parts, among them J2 J2_OUT, J3 Proto_GND, J4 Proto_1, J5 Proto_2, Q1 SI4894BDY, Q2 DMP3099L, U1 LTC1871EMS-7-PBF

Commit message: Auto-sync from Fortune at 2026-04-13 22:49:59
Routing:
- net GND: track 0.00 -> 64.1 mm, vias 0 -> 24

Commit message: Auto-sync from Fortune at 2026-04-13 23:12:01
Parts:
- J3, J4, J5: moved to F.Cu
- moved J3 8.25 mm to (133.0, 116.0)
- moved J5 8.18 mm to (133.0, 111.5)
- moved J4 8.02 mm to (133.0, 106.5)

Commit message: Auto-sync from Fortune at 2026-04-13 23:20:11
Parts:
- moved J3 9.50 mm to (133.0, 106.5)
- moved J4 5.00 mm to (133.0, 111.5)
- moved J5 4.50 mm to (133.0, 116.0)
Changed lines of the file:
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@@
 	(footprint "Connector_PinHeader_2.54mm:PinHeader_1x05_P2.54mm_Vertical"
 		(layer "F.Cu")
-		(at 133 111.5 -90)
+		(at 133 116 -90)
 		(descr "Through hole straight pin header, 1x05, 2.54mm pitch, single row")
 		(tags "Through hole pin header THT 1x05 2.54mm single row")
 		(property "Reference" "J5"
-			(at 0 -2.38 -90)
+			(at 0 -2.38 270)
 			(layer "F.SilkS")
 			(effects
@@
 		)
 		(property "Value" "Proto_2"
-			(at -2.5 9.46 180)
+			(at -2.5 9 180)
 			(layer "F.Fab")
 			(effects
@@
 	(footprint "Connector_PinHeader_2.54mm:PinHeader_1x05_P2.54mm_Vertical"
 		(layer "F.Cu")
-		(at 133 116 -90)
+		(at 133 106.5 -90)
 		(descr "Through hole straight pin header, 1x05, 2.54mm pitch, single row")
 		(tags "Through hole pin header THT 1x05 2.54mm single row")
 		(property "Reference" "J3"
-			(at 0 -2.38 -90)
+			(at 0 -2.38 270)
 			(layer "F.SilkS")
 			(effects
@@
 		)
 		(property "Value" "Proto_GND"
-			(at -2.5 8.5 180)
+			(at -2.5 8 180)
 			(layer "F.Fab")
 			(effects
@@
 	(footprint "Connector_PinHeader_2.54mm:PinHeader_1x05_P2.54mm_Vertical"
 		(layer "F.Cu")
-		(at 133 106.5 -90)
+		(at 133 111.5 -90)
 		(descr "Through hole straight pin header, 1x05, 2.54mm pitch, single row")
 		(tags "Through hole pin header THT 1x05 2.54mm single row")
 		(property "Reference" "J4"
-			(at 0 -2.38 -90)
+			(at 0 -2.38 270)
 			(layer "F.SilkS")
 			(effects
@@
 		)
 		(property "Value" "Proto_1"
-			(at -2.5 8.5 180)
+			(at -2.5 9 180)
 			(layer "F.Fab")
 			(effects

Commit message: Auto-sync from Fortune at 2026-04-14 15:01:52
Parts:
- moved J3 5.00 mm to (133.0, 111.5)
- moved J4 5.00 mm to (133.0, 106.5)
Routing:
- net Net-(D1-A): track 0.00 -> 169.7 mm
- net Net-(J4-Pin_2): track 0.00 -> 89.3 mm
- net Net-(U1-FB): track 0.00 -> 56.9 mm
- net Net-(D1-K): track 0.00 -> 50.6 mm
- net Net-(D2-K): track 0.00 -> 9.00 mm
- net Net-(U1-RUN): track 0.00 -> 8.84 mm
- net Net-(Q1-G): track 0.00 -> 7.95 mm
- net Net-(C2-Pad1): track 0.00 -> 7.07 mm
- net Net-(U1-FREQ): track 0.00 -> 6.02 mm
- net Net-(D2-A): track 0.00 -> 5.23 mm
- net Net-(U1-INTVCC): track 0.00 -> 4.46 mm
- net GND: track 64.1 -> 63.7 mm, vias 24 -> 23
Other:
- board text added: "LTC1871 Boost Converter"
- board text added: "Name: Fortune Olose EE499 Final Year Project"
