File: KiCAD PCB Design/LTC1871 KiCAD PCB Revision/LTC1871_Based_Boost_Controller_V2.kicad_pcb (KiCad board)
At the start: 2 copper layers, 60.5 x 42.5 mm, 36 parts, among them J2 J2_OUT, J3 Proto_GND, J4 Proto_1, J5 Proto_2, Q1 SI4894BDY, Q2 DMP3099L, U1 LTC1871EMS-7-PBF

Commit message: Auto-sync from Fortune at 2026-04-15 19:20:39
Parts:
- removed C1a8: 22µ, Capacitor_SMD:C_1206_3216Metric
- removed C5, Cin1: 100µ, Capacitor_THT:CP_Radial_D8.0mm_P3.50mm
- removed C8: 220n, Capacitor_SMD:C_0805_2012Metric
- removed D2: 1N4148, Diode_SMD:D_SOD-323_HandSoldering
- C1: value 10n -> 100µ; footprint Capacitor_SMD:C_0805_2012Metric -> Capacitor_THT:CP_Radial_D8.0mm_P3.50mm
- D1: footprint Diode_THT:D_DO-201AD_P15.24mm_Horizontal -> Package_TO_SOT_THT:TO-220-2_Vertical
- moved C1b2 18.0 mm to (174.0, 97.5)
- moved C1 15.8 mm to (123.8, 90.0), turned to 0 degrees
- moved D1 15.2 mm to (171.0, 91.5), turned to 180 degrees
- moved C1b1 13.5 mm to (170.5, 97.5)
- moved J2 1.50 mm to (178.0, 99.5)
- moved Q1 0.80 mm to (159.7, 103.4)
- renumbered J4 to J3, J3 to J4
Connections:
- C1 pad 1: Net-(D2-K) -> Net-(J3-Pin_2)
- C1a1 pad 1: Net-(D1-A) -> Net-(D1-K)
- C1a2 pad 1: Net-(D1-A) -> Net-(D1-K)
- C1a3 pad 1: Net-(D1-A) -> Net-(D1-K)
- C1a4 pad 1: Net-(D1-A) -> Net-(D1-K)
- C1a5 pad 1: Net-(D1-A) -> Net-(D1-K)
- C1a6 pad 1: Net-(D1-A) -> Net-(D1-K)
- C1a7 pad 1: Net-(D1-A) -> Net-(D1-K)
- C1b1 pad 1: Net-(D1-A) -> Net-(D1-K)
- C1b2 pad 1: Net-(D1-A) -> Net-(D1-K)
- C3 pad 1: Net-(D2-K) -> Net-(U1-ITH)
- C6 pad 1: Net-(J4-Pin_2) -> Net-(J3-Pin_2)
- C7 pad 1: Net-(J4-Pin_2) -> Net-(J3-Pin_2)
- J2 pad 1: Net-(D1-A) -> Net-(D1-K)
- J3 pad 2: Net-(J4-Pin_2) -> Net-(J3-Pin_2)
- J5 pad 2: Net-(D1-A) -> Net-(D1-K)
- J_VIN1 pad 1: Net-(J4-Pin_2) -> Net-(J3-Pin_2)
- L1 pad 1: Net-(J4-Pin_2) -> Net-(J3-Pin_2)
- L1 pad 2: Net-(D1-K) -> Net-(D1-A)
- Q1 pad 1: Net-(Q1-G) -> GND
- Q1 pad 2: Net-(D1-K) -> GND
- Q1 pad 3: GND -> Net-(Q1-G)
- Q1 pad 4: Net-(D1-K) -> GND
- Q1 pad 5: Net-(D1-K) -> Net-(D1-A)
- Q1 pad 6: Net-(D1-K) -> Net-(D1-A)
- Q1 pad 7: Net-(D1-K) -> Net-(D1-A)
- Q1 pad 8: Net-(D1-K) -> Net-(D1-A)
- Q2 pad 2: Net-(J4-Pin_2) -> Net-(J3-Pin_2)
- Q2 pad 3: Net-(J4-Pin_2) -> Net-(J3-Pin_2)
- R3 pad 1: Net-(D1-A) -> Net-(D1-K)
- R4 pad 2: Net-(D2-K) -> Net-(U1-ITH)
- R5 pad 1: Net-(J4-Pin_2) -> Net-(J3-Pin_2)
- U1 pad 10: Net-(D1-K) -> Net-(D1-A)
- U1 pad 2: Net-(D2-A) -> Net-(U1-ITH)
- U1 pad 9: Net-(J4-Pin_2) -> Net-(J3-Pin_2)
Routing:
- net Net-(D1-A): track 169.7 -> 63.7 mm, vias 0 -> 2
- net Net-(J4-Pin_2): track 89.5 -> 0.00 mm
- net Net-(J3-Pin_2): track 0.00 -> 89.4 mm
- net Net-(D1-K): track 50.8 -> 138.0 mm
- net Net-(U1-ITH): track 0.00 -> 15.8 mm
- net Net-(D2-K): track 9.00 -> 0.00 mm
- net Net-(D2-A): track 5.23 -> 0.00 mm
- net Net-(C2-Pad1): track 7.07 -> 4.57 mm
- net Net-(U1-FB): track 56.9 -> 58.9 mm
- net Net-(Q1-G): track 7.95 -> 9.67 mm
- net GND: track 63.7 -> 62.1 mm, vias 23 -> 18

Commit message: Auto-sync from Fortune at 2026-04-18 21:09:09
Parts:
- added C5: 100µ, Capacitor_THT:CP_Radial_D8.0mm_P3.50mm, F.Cu at (169.0, 81.0)
- added R7: 10k, Resistor_SMD:R_0805_2012Metric, F.Cu at (162.5, 87.8)
Connections:
- Q2 pad 1: GND -> Net-(Q2-G)
Routing:
- net Net-(Q2-G): track 0.00 -> 18.9 mm, vias 0 -> 2
- net Net-(D1-K): track 138.0 -> 143.3 mm

Commit message: Auto-sync from Fortune at 2026-04-19 09:47:09
Parts:
- added D2: 1N5818, Diode_THT:D_DO-41_SOD81_P10.16mm_Horizontal, F.Cu at (133.4, 93.6)
Connections:
- C1 pad 1: Net-(J3-Pin_2) -> Net-(D2-A)
- C6 pad 1: Net-(J3-Pin_2) -> Net-(D2-A)
- C7 pad 1: Net-(J3-Pin_2) -> Net-(D2-A)
- J3 pad 2: Net-(J3-Pin_2) -> Net-(D2-A)
- J_VIN1 pad 1: Net-(J3-Pin_2) -> Net-(D2-A)
- L1 pad 1: Net-(J3-Pin_2) -> Net-(D2-A)
- Q2 pad 2: Net-(J3-Pin_2) -> Net-(D2-A)
- Q2 pad 3: Net-(J3-Pin_2) -> Net-(D2-K)
- R5 pad 1: Net-(J3-Pin_2) -> Net-(D2-A)
- U1 pad 9: Net-(J3-Pin_2) -> Net-(D2-A)
Routing:
- net Net-(D2-A): track 0.00 -> 107.5 mm, vias 0 -> 3
- net Net-(J3-Pin_2): track 89.4 -> 0.00 mm
- net Net-(D2-K): track 0.00 -> 22.2 mm, vias 0 -> 2
- net Net-(Q2-G): track 18.9 -> 24.7 mm, vias 2 -> 4
