File: KiCAD PCB Design/LTC1871 KiCAD PCB Revision/LTC1871_Based_Boost_Controller_V2.kicad_pcb (KiCad board)
At the start: 2 copper layers, 60.5 x 42.5 mm, 34 parts, among them J2 J2_OUT, J3 Proto_1, J4 Proto_GND, J5 Proto_2, Q1 SI4894BDY, Q2 DMP3099L, U1 LTC1871EMS-7-PBF

Commit message: Auto-sync from Fortune at 2026-04-23 08:24:03
Parts:
- added D3: BZX84, Package_TO_SOT_SMD:SOT-23, F.Cu at (150.5, 87.5)
- added Q4: Q_NPN_BEC, Package_TO_SOT_SMD:SOT-23, F.Cu at (144.0, 80.0)
- added R8: 10k, Resistor_SMD:R_0402_1005Metric, F.Cu at (147.5, 80.0)
- added R9: 10k, Resistor_SMD:R_0402_1005Metric, F.Cu at (139.5, 82.5)
Routing:
- net Net-(D3-A): track 0.00 -> 15.8 mm, vias 0 -> 3
- net Net-(Q4-C): track 8.84 -> 22.4 mm, vias 0 -> 2
- net Net-(D3-K): track 0.00 -> 7.19 mm, vias 0 -> 2
- net GND: track 62.1 -> 66.2 mm, vias 18 -> 20
- net Net-(D2-A): track 107.5 -> 111.0 mm
