File: KiCAD PCB Design/LTC1871 KiCAD PCB Revision/LTC1871_Based_Boost_Controller_V2.kicad_sch (KiCad schematic)
At the start: 36 parts, among them J2 J2_OUT, J3 Proto_GND, J4 Proto_1, J5 Proto_2, Q1 SI4894BDY, Q2 DMP3099L, U1 LTC1871EMS-7-PBF

Commit message: Auto-sync from Fortune at 2026-04-15 19:20:39
Parts:
- removed C1: 10n, Capacitor_SMD:C_0805_2012Metric, symbol Device:C
- removed C1a8: 22µ, Capacitor_SMD:C_1206_3216Metric, symbol Device:C
- removed C5, Cin1: 100µ, Capacitor_THT:CP_Radial_D8.0mm_P3.50mm, symbol Device:C_Polarized
- removed C8: 220n, Capacitor_SMD:C_0805_2012Metric, symbol Device:C
- removed D2: 1N4148, Diode_SMD:D_SOD-323_HandSoldering, symbol Device:D
- added C1: 100µ, Capacitor_THT:CP_Radial_D8.0mm_P3.50mm, symbol Device:C_Polarized
- D1: footprint Diode_THT:D_DO-201AD_P15.24mm_Horizontal -> Package_TO_SOT_THT:TO-220-2_Vertical
- renumbered J4 to J3, J3 to J4
Connections:
- net GND: now also Q1.1 (S), Q1.2 (Source), Q1.4 (Source), C1.2; no longer Q1.3 (S)
- net at C6.1, C7.1, J3.2 (Pin_2)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: now also C1.1
- net at C1a1.1, C1a2.1, C1a3.1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: now also D1.1 (K); no longer D1.2 (A)
- net at C3.1, R4.2: now also U1.2 (ITH)
- net at L1.2, Q1.5 (D), Q1.6 (Drain)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: now also D1.2 (A); no longer D1.1 (K), Q1.2 (D), Q1.4 (Drain)
- net at U1.7 (GATE): now also Q1.3 (G); no longer Q1.1 (G)
Other:
- moved on the sheet: C1b1, C1b2, C7, D1, J3, J4

Commit message: Auto-sync from Fortune at 2026-04-18 21:09:09
Parts:
- added C5: 100µ, Capacitor_THT:CP_Radial_D8.0mm_P3.50mm, symbol Device:C_Polarized
- added R7: 10k, Resistor_SMD:R_0805_2012Metric, symbol Device:R
Connections:
- net GND: now also C5.2, R7.2; no longer Q2.1 (G)
- net at C1a1.1, C1a2.1, C1a3.1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: now also C5.1
- new net: Q2.1 (G), R7.1

Commit message: Auto-sync from Fortune at 2026-04-19 09:47:09
Parts:
- added D2: 1N5818, Diode_THT:D_DO-41_SOD81_P10.16mm_Horizontal, symbol Device:D_Schottky
Connections:
- net at C1.1, C6.1, C7.1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: now also D2.2 (A); no longer Q2.3 (D)
- new net: D2.1 (K), Q2.3 (D)
Changed lines of the file:
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@@
 	)
 	(junction
-		(at 146.05 55.88)
+		(at 82.55 33.02)
 		(diameter 0)
 		(color 0 0 0 0)
 	)
 	(junction
-		(at 82.55 33.02)
+		(at 146.05 55.88)
 		(diameter 0)
 		(color 0 0 0 0)
@@
 	(wire
 		(pts
-			(xy 146.05 55.88) (xy 147.32 55.88)
+			(xy 110.49 55.88) (xy 146.05 55.88)
 		)
 		(stroke
@@
 	(wire
 		(pts
+			(xy 146.05 52.07) (xy 146.05 55.88)
+		)
+		(stroke
+			(width 0)
+			(type default)
+		)
+	)
+	(wire
+		(pts
 			(xy 76.2 33.02) (xy 76.2 38.1)
 		)
@@
 	(wire
 		(pts
-			(xy 110.49 55.88) (xy 146.05 55.88)
-		)
-		(stroke
-			(width 0)
-			(type default)
-		)
-	)
-	(wire
-		(pts
 			(xy 110.49 55.88) (xy 110.49 30.48)
 		)
@@
 	(wire
 		(pts
+			(xy 146.05 55.88) (xy 147.32 55.88)
+		)
+		(stroke
+			(width 0)
+			(type default)
+		)
+	)
+	(wire
+		(pts
 			(xy 198.12 104.14) (xy 198.12 111.76)
 		)
@@
 	(wire
 		(pts
-			(xy 146.05 41.91) (xy 146.05 55.88)
-		)
-		(stroke
-			(width 0)
-			(type default)
-		)
-	)
-	(wire
-		(pts
 			(xy 142.24 96.52) (xy 142.24 100.33)
 		)
@@
 	(wire
 		(pts
+			(xy 146.05 41.91) (xy 146.05 44.45)
+		)
+		(stroke
+			(width 0)
+			(type default)
+		)
+	)
+	(wire
+		(pts
 			(xy 68.58 95.25) (xy 68.58 93.98)
 		)
@@
 					(unit 1)
 				)
+			)
+		)
+	)
+	(symbol
+		(lib_id "Device:D_Schottky")
+		(at 146.05 48.26 270)
+		(unit 1)
+		(body_style 1)
+		(exclude_from_sim no)
+		(in_bom yes)
+		(on_board yes)
+		(in_pos_files yes)
+		(dnp no)
+		(property "Reference" "D2"
+			(at 148.59 46.6724 90)
+			(show_name no)
+			(do_not_autoplace no)
+			(effects
+				(font
+					(size 1.27 1.27)
+				)
+				(justify left)
+			)
+		)
+		(property "Value" "1N5818"
+			(at 148.59 48.514 90)
+			(show_name no)
+			(do_not_autoplace no)
+			(effects
+				(font
+					(size 1.27 1.27)
+				)
+				(justify left)
+			)
+		)
+		(property "Footprint" "Diode_THT:D_DO-41_SOD81_P10.16mm_Horizontal"
+			(at 146.05 48.26 0)
+			(hide yes)
+			(show_name no)
+			(do_not_autoplace no)
+			(effects
+				(font
+					(size 1.27 1.27)
+				)
+			)
+		)
+		(property "Datasheet" ""
+			(at 146.05 48.26 0)
+			(hide yes)
+			(show_name no)
+			(do_not_autoplace no)
+			(effects
+				(font
+					(size 1.27 1.27)
+				)
+			)
+		)
+		(property "Description" "Schottky diode"
+			(at 146.05 48.26 0)
+			(hide yes)
+			(show_name no)
+			(do_not_autoplace no)
+			(effects
+				(font
+					(size 1.27 1.27)
+				)
+			)
+		)
+		(pin "2"
+		)
+		(pin "1"
+		)
+		(instances
+			(project "LTC1871_Based_Boost_Controller_V2"
+				(path "/afd51646-14c5-4e75-88ba-419bc48b66e0"
+					(reference "D2")
+					(unit 1)
+				)

Commit message: Auto-sync from EECR-HN3V674 at 2026-04-22 19:15:57
Parts:
- added D3: D_Zener, symbol Device:D_Zener
- added Q3: Q_Dual_NPN_NPN_B1E2B2C2E1C1, symbol Transistor_BJT:Q_Dual_NPN_NPN_B1E2B2C2E1C1
- added R8, R9: R, symbol Device:R
Connections:
- net GND: now also Q3.5 (E1), R9.2
- net at C1.1, C6.1, C7.1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: now also R8.1
- net at R5.2, R6.1, U1.1 (RUN): now also Q3.6 (C1)
- new net: D3.2 (A), Q3.1 (B1), R9.1
- new net: D3.1 (K), R8.2

Commit message: Auto-sync from Fortune at 2026-04-23 00:30:17
Parts:
- removed Q3: Q_Dual_NPN_NPN_B1E2B2C2E1C1, symbol Transistor_BJT:Q_Dual_NPN_NPN_B1E2B2C2E1C1
- added Q4: Q_NPN_BEC, Package_TO_SOT_SMD:SOT-23, symbol Transistor_BJT:Q_NPN_BEC
- D3: value D_Zener -> BZX84; footprint (none) -> Package_TO_SOT_SMD:SOT-23
- R8, R9: value R -> 10k; footprint (none) -> Package_TO_SOT_SMD:SOT-23
Connections:
- net GND: now also Q4.2 (E)
- net at D3.2 (A), R9.1: now also Q4.1 (B)
- net at R5.2, R6.1, U1.1 (RUN): now also Q4.3 (C)
Changed lines of the file:
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@@
 	)
 	(junction
-		(at 138.43 17.78)
-		(diameter 0)
-		(color 0 0 0 0)
-	)
-	(junction
 		(at 214.63 86.36)
 		(diameter 0)
@@
 	)
 	(junction
+		(at 138.43 17.78)
+		(diameter 0)
+		(color 0 0 0 0)
+	)
+	(junction
 		(at 147.32 66.04)
 		(diameter 0)
@@
 	(wire
 		(pts
-			(xy 185.42 12.7) (xy 185.42 7.62)
-		)
-		(stroke
-			(width 0)
-			(type default)
-		)
-	)
-	(wire
-		(pts
 			(xy 76.2 38.1) (xy 82.55 38.1)
 		)
@@
 	(wire
 		(pts
-			(xy 185.42 22.86) (xy 185.42 36.83)
+			(xy 184.15 22.86) (xy 184.15 25.4)
 		)
 		(stroke
@@
 	(wire
 		(pts
-			(xy 185.42 7.62) (xy 160.02 7.62)
+			(xy 184.15 12.7) (xy 160.02 12.7)
 		)
 		(stroke
@@
 	(wire
 		(pts
+			(xy 184.15 25.4) (xy 185.42 25.4)
+		)
+		(stroke
+			(width 0)
+			(type default)
+		)
+	)
+	(wire
+		(pts
 			(xy 173.99 96.52) (xy 176.53 96.52)
 		)
@@
 	(wire
 		(pts
+			(xy 185.42 25.4) (xy 185.42 36.83)
+		)
+		(stroke
+			(width 0)
+			(type default)
+		)
+	)
+	(wire
+		(pts
 			(xy 111.76 41.91) (xy 111.76 35.56)
 		)
@@
 	(wire
 		(pts
-			(xy 138.43 17.78) (xy 177.8 17.78)
+			(xy 138.43 17.78) (xy 176.53 17.78)
 		)
 		(stroke
@@
 	(wire
 		(pts
-			(xy 160.02 7.62) (xy 160.02 60.96)
+			(xy 160.02 12.7) (xy 160.02 60.96)
 		)
 		(stroke
@@
 	)
 	(symbol
-		(lib_id "Transistor_BJT:Q_Dual_NPN_NPN_B1E2B2C2E1C1")
-		(at 182.88 17.78 0)
-		(unit 1)
-		(body_style 1)
-		(exclude_from_sim no)
-		(in_bom yes)
-		(on_board yes)
-		(in_pos_files yes)
-		(dnp no)
-		(property "Reference" "Q3"
-			(at 187.96 16.5099 0)
-			(show_name no)
-			(do_not_autoplace no)
-			(effects
-				(font
-					(size 1.27 1.27)
-				)
-				(justify left)
-			)
-		)
-		(property "Value" "Q_Dual_NPN_NPN_B1E2B2C2E1C1"
-			(at 181.61 24.892 0)
-			(show_name no)
-			(do_not_autoplace no)
-			(effects
-				(font
-					(size 1.27 1.27)
-				)
-				(justify left)
-			)
-		)
-		(property "Footprint" ""
-			(at 187.96 15.24 0)
-			(hide yes)
-			(show_name no)
-			(do_not_autoplace no)
-			(effects
-				(font
-					(size 1.27 1.27)
-				)
-			)
-		)
-		(property "Datasheet" ""
-			(at 182.88 17.78 0)
-			(hide yes)
-			(show_name no)
-			(do_not_autoplace no)
-			(effects
-				(font
-					(size 1.27 1.27)
-				)
-			)
-		)
-		(property "Description" "Dual NPN transistor, 6 pin package"
-			(at 182.88 17.78 0)
-			(hide yes)
-			(show_name no)
-			(do_not_autoplace no)
-			(effects
-				(font
-					(size 1.27 1.27)
-				)
-			)
-		)
-		(pin "1"
-		)
-		(pin "6"
-		)
-		(pin "2"
-		)
-		(pin "5"
-		)
-		(pin "3"
-		)
-		(pin "4"
-		)
-		(instances
-			(project "LTC1871_Based_Boost_Controller_V2"
-				(path "/afd51646-14c5-4e75-88ba-419bc48b66e0"
-					(reference "Q3")
-					(unit 1)
-				)
-			)
-		)
-	)
-	(symbol
 		(lib_id "power:GND")
 		(at 157.48 90.17 90)
@@
 			)
 		)
-		(property "Value" "D_Zener"
+		(property "Value" "BZX84"
 			(at 123.19 13.97 0)
 			(show_name no)
@@
 			)
 		)
-		(property "Footprint" ""
+		(property "Footprint" "Package_TO_SOT_SMD:SOT-23"
 			(at 123.19 17.78 0)
 			(hide yes)
@@
 			)
 		)
-		(property "Value" "R"
+		(property "Value" "10k"
 			(at 140.97 26.6699 0)
 			(show_name no)
@@
 			)
 		)
-		(property "Footprint" ""
+		(property "Footprint" "Package_TO_SOT_SMD:SOT-23"
 			(at 136.652 25.4 90)
 			(hide yes)
@@
 			)
 		)
-		(property "Value" "R"
+		(property "Value" "10k"
 			(at 111.76 13.97 90)
 			(show_name no)
@@
 			)
 		)
-		(property "Footprint" ""
+		(property "Footprint" "Package_TO_SOT_SMD:SOT-23"
 			(at 111.76 19.558 90)
 			(hide yes)
@@
 					(unit 1)
 				)
+			)
+		)
+	)
+	(symbol
+		(lib_id "Transistor_BJT:Q_NPN_BEC")
+		(at 181.61 17.78 0)
+		(unit 1)
+		(body_style 1)
+		(exclude_from_sim no)
+		(in_bom yes)
+		(on_board yes)
+		(in_pos_files yes)
+		(dnp no)
+		(fields_autoplaced yes)
+		(property "Reference" "Q4"
+			(at 186.69 16.5099 0)
+			(show_name no)
+			(do_not_autoplace no)
+			(effects
+				(font
+					(size 1.27 1.27)
+				)
+				(justify left)
+			)
+		)
+		(property "Value" "Q_NPN_BEC"
+			(at 186.69 19.0499 0)
+			(show_name no)
+			(do_not_autoplace no)
+			(effects
+				(font
+					(size 1.27 1.27)
+				)
+				(justify left)
+			)
+		)
+		(property "Footprint" "Package_TO_SOT_SMD:SOT-23"
+			(at 186.69 15.24 0)
+			(hide yes)
+			(show_name no)
+			(do_not_autoplace no)
+			(effects
+				(font
+					(size 1.27 1.27)
+				)
+			)
+		)
+		(property "Datasheet" ""
+			(at 181.61 17.78 0)
+			(hide yes)
+			(show_name no)
+			(do_not_autoplace no)
+			(effects
+				(font
+					(size 1.27 1.27)
+				)
+			)
+		)
+		(property "Description" "NPN transistor, base/emitter/collector"
+			(at 181.61 17.78 0)
+			(hide yes)
+			(show_name no)
+			(do_not_autoplace no)
+			(effects
+				(font
+					(size 1.27 1.27)
+				)
+			)
+		)
+		(property "Sim.Device" "NPN"
+			(at 181.61 17.78 0)
+			(hide yes)
+			(show_name no)
+			(do_not_autoplace no)
+			(effects
+				(font
+					(size 1.27 1.27)
+				)
+			)
+		)
+		(property "Sim.Pins" "1=B 2=E 3=C"
+			(at 181.61 17.78 0)
+			(hide yes)
+			(show_name no)
+			(do_not_autoplace no)
+			(effects
+				(font
+					(size 1.27 1.27)
+				)
+			)
+		)
+		(pin "1"
+		)
+		(pin "2"
+		)
+		(pin "3"
+		)
+		(instances
+			(project "LTC1871_Based_Boost_Controller_V2"
+				(path "/afd51646-14c5-4e75-88ba-419bc48b66e0"
+					(reference "Q4")
+					(unit 1)
+				)
