File: KiCAD PCB Design/LTC1871 KiCAD PCB Revision/LTC1871_Based_Boost_Controller_V2 - Copy.kicad_pcb (KiCad board)
At the start: 2 copper layers, 60.5 x 42.5 mm, 38 parts, among them J2 J2_OUT, J3 Proto_1, J4 Proto_GND, J5 Proto_2, Q1 SI4894BDY, Q2 DMP3099L, Q4 Q_NPN_BEC, U1 LTC1871EMS-7-PBF

Commit message: Auto-sync from Fortune at 2026-05-06 01:04:25
Parts:
- R5: value 549k -> 49k
- R6: value 100K -> 10K
Changed lines of the file:
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@@
 			)
 		)
-		(property "Value" "549k"
+		(property "Value" "49k"
 			(at 0.0875 1.5 90)
 			(layer "F.Fab")
@@
 			)
 		)
-		(property "Value" "100K"
+		(property "Value" "10K"
 			(at 0 1.65 90)
 			(layer "F.Fab")

Commit message: Auto-sync from Fortune at 2026-05-07 01:50:28
Parts:
- D2: value 1N5818 -> SS14; footprint Diode_THT:D_DO-41_SOD81_P10.16mm_Horizontal -> Diode_SMD:D_SMA
- R8: value 10k -> 5.38k
- moved D2 2.13 mm to (135.5, 93.5)
Routing:
- net Net-(D2-A): track 111.0 -> 117.0 mm
Changed lines of the file:
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@@
 		(aux_axis_origin 120.239892 118.379686)
 		(pcbplotparams
-			(layerselection 0x00000000_00000000_55555555_5755f5ff)
+			(layerselection 0x00000000_00000000_55555555_575575ff)
 			(plot_on_all_layers_selection 0x00000000_00000000_00000000_00000000)
 			(disableapertmacros no)
-			(usegerberextensions no)
+			(usegerberextensions yes)
 			(usegerberattributes yes)
 			(usegerberadvancedattributes yes)
@@
 		(tags "capacitor")
 		(property "Reference" "C3"
-			(at -2.45 0 0)
+			(at 0.55 -2 0)
 			(layer "F.SilkS")
 			(effects
@@
 		(tags "resistor")
 		(property "Reference" "R5"
-			(at 0 2 90)
+			(at -1.4125 3.5 90)
 			(layer "F.SilkS")
 			(effects
@@
 		)
 		(property "Value" "49k"
-			(at 0.0875 1.5 90)
+			(at 0.0875 2 90)
 			(layer "F.Fab")
 			(effects
@@
 		)
 		(property "Value" "22µ"
-			(at 3.4 -0.025 0)
+			(at 3 0 0)
 			(layer "F.Fab")
 			(effects
@@
 			)
 		)
-		(property "Value" "10k"
+		(property "Value" "5.38k"
 			(at 0 1.17 0)
 			(layer "F.Fab")
@@
 		)
 	)
-	(footprint "Diode_THT:D_DO-41_SOD81_P10.16mm_Horizontal"
+	(footprint "Diode_SMD:D_SMA"
 		(layer "F.Cu")
-		(at 133.375 93.625)
-		(descr "Diode, DO-41_SOD81 series, Axial, Horizontal, pin pitch=10.16mm, length*diameter=5.2*2.7mm^2, https://www.diodes.com/assets/Package-Files/DO-41-Plastic.pdf")
-		(tags "Diode DO-41_SOD81 series Axial Horizontal pin pitch 10.16mm  length 5.2mm diameter 2.7mm")
+		(at 135.5 93.5)
+		(descr "Diode SMA (DO-214AC)")
+		(tags "Diode SMA (DO-214AC)")
 		(property "Reference" "D2"
-			(at 5.08 -2.47 0)
+			(at 0 -2.5 0)
 			(layer "F.SilkS")
 			(effects
@@
 			)
 		)
-		(property "Value" "1N5818"
-			(at 5.08 2.47 0)
+		(property "Value" "SS14"
+			(at 5 1.5 0)
 			(layer "F.Fab")
 			(effects
@@
 		(property "Datasheet" ""
 			(at 0 0 0)
+			(unlocked yes)
 			(layer "F.Fab")
 			(hide yes)
@@
 				(font
 					(size 1.27 1.27)
+					(thickness 0.15)
 				)
 			)
@@
 		(property "Description" "Schottky diode"
 			(at 0 0 0)
+			(unlocked yes)
 			(layer "F.Fab")
 			(hide yes)
@@
 				(font
 					(size 1.27 1.27)
-				)
-			)
-		)
-		(property "KiLib_Generator" "diode/THT"
-			(at 0 0 0)
-			(layer "F.SilkS")
-			(hide yes)
-			(effects
-				(font
-					(size 1 1)
 					(thickness 0.15)
 				)
@@
 			)
 		)
-		(attr through_hole)
+		(attr smd)
 		(duplicate_pad_numbers_are_jumpers no)
 		(fp_line
-			(start 1.34 0)
-			(end 2.36 0)
+			(start -3.51 -1.65)
+			(end -3.51 1.65)
 			(stroke
 				(width 0.12)
@@
 		)
 		(fp_line
-			(start 3.14 -1.47)
-			(end 3.14 1.47)
+			(start -3.51 -1.65)
+			(end 2 -1.65)
 			(stroke
 				(width 0.12)
@@
 		)
 		(fp_line
-			(start 3.26 -1.47)
-			(end 3.26 1.47)
+			(start -3.51 1.65)
+			(end 2 1.65)
 			(stroke
 				(width 0.12)
@@
 		)
 		(fp_line
-			(start 3.38 -1.47)
-			(end 3.38 1.47)
+			(start -3.5 -1.75)
+			(end 3.5 -1.75)
 			(stroke
-				(width 0.12)
+				(width 0.05)
 				(type solid)
 			)
-			(layer "F.SilkS")
+			(layer "F.CrtYd")
 		)
 		(fp_line
-			(start 8.82 0)
-			(end 7.8 0)
+			(start -3.5 1.75)
+			(end -3.5 -1.75)
 			(stroke
-				(width 0.12)
+				(width 0.05)
 				(type solid)
 			)
-			(layer "F.SilkS")
+			(layer "F.CrtYd")
 		)
-		(fp_rect
-			(start 2.36 -1.47)
-			(end 7.8 1.47)
+		(fp_line
+			(start 3.5 -1.75)
+			(end 3.5 1.75)
 			(stroke
-				(width 0.12)
+				(width 0.05)
 				(type solid)
 			)
-			(fill no)
-			(layer "F.SilkS")
+			(layer "F.CrtYd")
 		)
-		(fp_rect
-			(start -1.35 -1.6)
-			(end 11.51 1.6)
+		(fp_line
+			(start 3.5 1.75)
+			(end -3.5 1.75)
 			(stroke
 				(width 0.05)
 				(type solid)
 			)
-			(fill no)
 			(layer "F.CrtYd")
 		)
 		(fp_line
-			(start 0 0)
-			(end 2.48 0)
+			(start -2.3 1.5)
+			(end -2.3 -1.5)
 			(stroke
 				(width 0.1)
@@
 		)
 		(fp_line
-			(start 3.16 -1.35)
-			(end 3.16 1.35)
+			(start -0.64944 -0.79908)
+			(end -0.64944 0.80112)
 			(stroke
 				(width 0.1)
@@
 		)
 		(fp_line
-			(start 3.26 -1.35)
-			(end 3.26 1.35)
+			(start -0.64944 0.00102)
+			(end -1.55114 0.00102)
 			(stroke
 				(width 0.1)
@@
 		)
 		(fp_line
-			(start 3.36 -1.35)
-			(end 3.36 1.35)
+			(start -0.64944 0.00102)
+			(end 0.50118 -0.79908)
 			(stroke
 				(width 0.1)
@@
 		)
 		(fp_line
-			(start 10.16 0)
-			(end 7.68 0)
+			(start -0.64944 0.00102)
+			(end 0.50118 0.75032)
 			(stroke
 				(width 0.1)
@@
 			(layer "F.Fab")
 		)
-		(fp_rect
-			(start 2.48 -1.35)
-			(end 7.68 1.35)
+		(fp_line
+			(start 0.50118 0.00102)
+			(end 1.4994 0.00102)
 			(stroke
 				(width 0.1)
 				(type solid)
 			)
-			(fill no)
 			(layer "F.Fab")
 		)
-		(fp_text user "K"
-			(at 0 -2.1 0)
-			(layer "F.SilkS")
-			(effects
-				(font
-					(size 1 1)
-					(thickness 0.15)
-				)
+		(fp_line
+			(start 0.50118 0.75032)
+			(end 0.50118 -0.79908)
+			(stroke
+				(width 0.1)
+				(type solid)
 			)
+			(layer "F.Fab")
 		)
-		(fp_text user "K"
-			(at 0 -2.1 0)
+		(fp_line
+			(start 2.3 -1.5)
+			(end -2.3 -1.5)
+			(stroke
+				(width 0.1)
+				(type solid)
+			)
 			(layer "F.Fab")
-			(effects
-				(font
-					(size 1 1)
-					(thickness 0.15)
-				)
+		)
+		(fp_line
+			(start 2.3 -1.5)
+			(end 2.3 1.5)
+			(stroke
+				(width 0.1)
+				(type solid)
 			)
+			(layer "F.Fab")
+		)
+		(fp_line
+			(start 2.3 1.5)
+			(end -2.3 1.5)
+			(stroke
+				(width 0.1)
+				(type solid)
+			)
+			(layer "F.Fab")
 		)
 		(fp_text user "${REFERENCE}"
-			(at 5.47 0 0)
+			(at 0 -2.5 0)
 			(layer "F.Fab")
 			(effects
@@
 			)
 		)
-		(pad "1" thru_hole roundrect
-			(at 0 0)
-			(size 2.2 2.2)
-			(drill 1.1)
-			(layers "*.Cu" "*.Mask")
-			(remove_unused_layers no)
-			(roundrect_rratio 0.113636)
+		(pad "1" smd roundrect
+			(at -2 0)
+			(size 2.5 1.8)
+			(layers "F.Cu" "F.Mask" "F.Paste")
+			(roundrect_rratio 0.1388888889)
 			(net "Net-(D2-K)")
 			(pinfunction "K_1")
 			(pintype "passive")
 		)
-		(pad "2" thru_hole circle
-			(at 10.16 0)
-			(size 2.2 2.2)
-			(drill 1.1)
-			(layers "*.Cu" "*.Mask")
-			(remove_unused_layers no)
+		(pad "2" smd roundrect
+			(at 2 0)
+			(size 2.5 1.8)
+			(layers "F.Cu" "F.Mask" "F.Paste")
+			(roundrect_rratio 0.1388888889)
 			(net "Net-(D2-A)")
 			(pinfunction "A_2")
@@
 		)
 		(embedded_fonts no)
-		(model "${KICAD10_3DMODEL_DIR}/Diode_THT.3dshapes/D_DO-41_SOD81_P10.16mm_Horizontal.step"
+		(model "${KICAD10_3DMODEL_DIR}/Diode_SMD.3dshapes/D_SMA.step"
 			(offset
 				(xyz 0 0 0)
@@
 		)
 		(property "Value" "22µ"
-			(at 3.4 -0.175 0)
+			(at 0 -2.65 0)
 			(layer "F.Fab")
 			(effects
@@
 	)
 	(segment
+		(start 143.41 93.5)
+		(end 137.5 93.5)
+		(width 1)
+		(layer "F.Cu")
+		(net "Net-(D2-A)")
+	)
+	(segment
 		(start 132 83.5)
 		(end 132 86.525)
@@
 	)
 	(segment
+		(start 143.535 93.625)
+		(end 143.41 93.5)
+		(width 1)
+		(layer "F.Cu")
+		(net "Net-(D2-A)")
+	)
+	(segment
 		(start 132 86.525)
 		(end 135.35 86.525)
@@
 	)
 	(segment
-		(start 133.375 93.625)
-		(end 133.375 95.875)
-		(width 0.5)
-		(layer "F.Cu")
-		(net "Net-(D2-K)")
-	)
-	(segment
-		(start 133.375 95.875)
-		(end 133.5 96)
+		(start 133.5 96)
+		(end 133.5 93.5)
 		(width 0.5)
 		(layer "F.Cu")
