File: KiCAD PCB Design/LTC1871 KiCAD PCB Revision/LTC1871_Based_Boost_Controller_V2 - Copy.kicad_sch (KiCad schematic)
At the start: 38 parts, among them J2 J2_OUT, J3 Proto_1, J4 Proto_GND, J5 Proto_2, Q1 SI4894BDY, Q2 DMP3099L, Q4 Q_NPN_BEC, U1 LTC1871EMS-7-PBF

Commit message: Auto-sync from Fortune at 2026-04-24 18:05:31
Parts:
- R5: value 549k -> 49k
- R6: value 100K -> 10K
- R8: value 10k -> 5.38k

Commit message: Auto-sync from Fortune at 2026-04-26 07:34:23
Parts:
- R5: value 49k -> 549k
- R6: value 10K -> 100K
- R8: value 5.38k -> 10k; footprint Package_TO_SOT_SMD:SOT-23 -> Resistor_SMD:R_0402_1005Metric
- R9: footprint Package_TO_SOT_SMD:SOT-23 -> Resistor_SMD:R_0402_1005Metric
Changed lines of the file:
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@@
 			)
 		)
-		(property "Value" "49k"
+		(property "Value" "549k"
 			(at 106.68 43.1799 0)
 			(show_name no)
@@
 			)
 		)
-		(property "Footprint" "Package_TO_SOT_SMD:SOT-23"
+		(property "Footprint" "Resistor_SMD:R_0402_1005Metric"
 			(at 136.652 25.4 90)
 			(hide yes)
@@
 			)
 		)
-		(property "Value" "5.38k"
+		(property "Value" "10k"
 			(at 111.76 13.97 90)
 			(show_name no)
@@
 			)
 		)
-		(property "Footprint" "Package_TO_SOT_SMD:SOT-23"
+		(property "Footprint" "Resistor_SMD:R_0402_1005Metric"
 			(at 111.76 19.558 90)
 			(hide yes)
@@
 			)
 		)
-		(property "Value" "10K"
+		(property "Value" "100K"
 			(at 106.68 53.3399 0)
 			(show_name no)

Commit message: Auto-sync from Fortune at 2026-05-05 08:49:35
Parts:
- R5: value 549k -> 49k
- R6: value 100K -> 10K
Changed lines of the file:
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@@
 		(in_pos_files yes)
 		(dnp no)
-		(fields_autoplaced yes)
 		(property "Reference" "D3"
-			(at 123.19 11.43 0)
+			(at 123.19 14.986 0)
 			(show_name no)
 			(do_not_autoplace no)
@@
 		)
 		(property "Value" "BZX84"
-			(at 123.19 13.97 0)
+			(at 123.19 20.574 0)
 			(show_name no)
 			(do_not_autoplace no)
@@
 		(in_pos_files yes)
 		(dnp no)
-		(fields_autoplaced yes)
 		(property "Reference" "#PWR026"
 			(at 104.14 64.77 0)
@@
 		)
 		(property "Value" "GND"
-			(at 104.14 63.5 0)
+			(at 104.14 62.23 0)
 			(show_name no)
 			(do_not_autoplace no)
@@
 		(in_pos_files yes)
 		(dnp no)
-		(fields_autoplaced yes)
 		(property "Reference" "R7"
-			(at 128.27 24.13 90)
+			(at 128.524 32.766 90)
 			(show_name no)
 			(do_not_autoplace no)
@@
 		)
 		(property "Value" "10k"
-			(at 128.27 26.67 90)
+			(at 128.524 28.194 90)
 			(show_name no)
 			(do_not_autoplace no)
@@
 		(in_pos_files yes)
 		(dnp no)
-		(fields_autoplaced yes)
 		(property "Reference" "R5"
-			(at 106.68 40.6399 0)
+			(at 102.108 43.434 90)
 			(show_name no)
 			(do_not_autoplace no)
@@
 			)
 		)
-		(property "Value" "549k"
-			(at 106.68 43.1799 0)
+		(property "Value" "49k"
+			(at 106.426 43.942 90)
 			(show_name no)
 			(do_not_autoplace no)
@@
 		(dnp no)
 		(property "Reference" "D2"
-			(at 148.59 46.6724 90)
+			(at 143.51 47.244 0)
 			(show_name no)
 			(do_not_autoplace no)
@@
 		)
 		(property "Value" "1N5818"
-			(at 148.59 48.514 90)
+			(at 148.844 44.958 0)
 			(show_name no)
 			(do_not_autoplace no)
@@
 		(in_pos_files yes)
 		(dnp no)
-		(fields_autoplaced yes)
 		(property "Reference" "R9"
-			(at 140.97 24.1299 0)
+			(at 134.366 25.4 0)
 			(show_name no)
 			(do_not_autoplace no)
@@
 		)
 		(property "Value" "10k"
-			(at 140.97 26.6699 0)
+			(at 140.208 25.146 0)
 			(show_name no)
 			(do_not_autoplace no)
@@
 		(in_pos_files yes)
 		(dnp no)
-		(fields_autoplaced yes)
 		(property "Reference" "R8"
-			(at 111.76 11.43 90)
+			(at 111.76 20.32 90)
 			(show_name no)
 			(do_not_autoplace no)
@@
 		)
 		(property "Value" "10k"
-			(at 111.76 13.97 90)
+			(at 111.76 15.24 90)
 			(show_name no)
 			(do_not_autoplace no)
@@
 		(in_pos_files yes)
 		(dnp no)
-		(fields_autoplaced yes)
 		(property "Reference" "R6"
-			(at 106.68 50.7999 0)
+			(at 102.108 53.34 90)
 			(show_name no)
 			(do_not_autoplace no)
@@
 			)
 		)
-		(property "Value" "100K"
-			(at 106.68 53.3399 0)
+		(property "Value" "10K"
+			(at 106.172 54.356 90)
 			(show_name no)
 			(do_not_autoplace no)
@@
 		(in_pos_files yes)
 		(dnp no)
-		(fields_autoplaced yes)
 		(property "Reference" "Q4"
-			(at 186.69 16.5099 0)
+			(at 179.07 13.97 0)
 			(show_name no)
 			(do_not_autoplace no)
@@
 		)
 		(property "Value" "Q_NPN_BEC"
-			(at 186.69 19.0499 0)
+			(at 182.88 34.29 90)
 			(show_name no)
 			(do_not_autoplace no)

Commit message: Auto-sync from Fortune at 2026-05-07 01:50:28
Parts:
- D2: value 1N5818 -> SS14; footprint Diode_THT:D_DO-41_SOD81_P10.16mm_Horizontal -> Diode_SMD:D_SMA
- R8: value 10k -> 5.38k
Changed lines of the file:
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@@
 			)
 		)
-		(property "Value" "1N5818"
+		(property "Value" "SS14"
 			(at 148.844 44.958 0)
 			(show_name no)
@@
 			)
 		)
-		(property "Footprint" "Diode_THT:D_DO-41_SOD81_P10.16mm_Horizontal"
+		(property "Footprint" "Diode_SMD:D_SMA"
 			(at 146.05 48.26 0)
 			(hide yes)
@@
 			)
 		)
-		(property "Value" "10k"
+		(property "Value" "5.38k"
 			(at 111.76 15.24 90)
 			(show_name no)
